File: thundermaus.brd (EAGLE design)
At the start: 120.6 x 74.9 mm, 46 parts, among them IC1 LM7805, IC2 TINY24/44/84-PU, Q1 FGH20N60SFD, Q2 2n7000, Q3 2n7000, X1 TOBU3

Commit message: merge v2 changes; drop D6, move few things subtly
Parts:
- removed D6: 1N5353, diode:C1702-15
Connections:
- new net N$2: D5.A, IC1.IN, R2.2
- net GND: no longer D5.A, D6.A, D6.C, IC1.IN, R2.2
Routing:
- net N$2: track 0.00 -> 13.0 mm
- net GND: track 51.1 -> 38.1 mm
Changed lines of the file:
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@@
 <grid distance="0.025" unitdist="inch" unit="inch" style="lines" multiple="4" display="yes" altdistance="0.0125" altunitdist="inch" altunit="inch"/>
 <layers>
-<layer number="1" name="Top" color="4" fill="1" visible="yes" active="yes"/>
+<layer number="1" name="Top" color="4" fill="1" visible="no" active="yes"/>
 <layer number="2" name="Route2" color="1" fill="3" visible="no" active="yes"/>
 <layer number="3" name="Route3" color="4" fill="3" visible="no" active="yes"/>
@@
 <layer number="14" name="Route14" color="1" fill="6" visible="no" active="yes"/>
 <layer number="15" name="Route15" color="4" fill="6" visible="no" active="yes"/>
-<layer number="16" name="Bottom" color="1" fill="1" visible="yes" active="yes"/>
+<layer number="16" name="Bottom" color="1" fill="1" visible="no" active="yes"/>
 <layer number="17" name="Pads" color="2" fill="1" visible="yes" active="yes"/>
 <layer number="18" name="Vias" color="2" fill="1" visible="yes" active="yes"/>
 <layer number="19" name="Unrouted" color="6" fill="1" visible="no" active="yes"/>
 <layer number="20" name="Dimension" color="15" fill="1" visible="yes" active="yes"/>
-<layer number="21" name="tPlace" color="7" fill="1" visible="no" active="yes"/>
-<layer number="22" name="bPlace" color="7" fill="1" visible="no" active="yes"/>
+<layer number="21" name="tPlace" color="7" fill="1" visible="yes" active="yes"/>
+<layer number="22" name="bPlace" color="7" fill="1" visible="yes" active="yes"/>
 <layer number="23" name="tOrigins" color="15" fill="1" visible="yes" active="yes"/>
-<layer number="24" name="bOrigins" color="15" fill="1" visible="no" active="yes"/>
-<layer number="25" name="tNames" color="7" fill="1" visible="no" active="yes"/>
-<layer number="26" name="bNames" color="7" fill="1" visible="no" active="yes"/>
-<layer number="27" name="tValues" color="7" fill="1" visible="no" active="yes"/>
-<layer number="28" name="bValues" color="7" fill="1" visible="no" active="yes"/>
+<layer number="24" name="bOrigins" color="15" fill="1" visible="yes" active="yes"/>
+<layer number="25" name="tNames" color="7" fill="1" visible="yes" active="yes"/>
+<layer number="26" name="bNames" color="7" fill="1" visible="yes" active="yes"/>
+<layer number="27" name="tValues" color="7" fill="1" visible="yes" active="yes"/>
+<layer number="28" name="bValues" color="7" fill="1" visible="yes" active="yes"/>
 <layer number="29" name="tStop" color="7" fill="3" visible="no" active="yes"/>
 <layer number="30" name="bStop" color="7" fill="6" visible="no" active="yes"/>
@@
 <attribute name="VALUE" x="68.58" y="6.35" size="1.27" layer="27"/>
 </element>
-<element name="D6" library="diode" package="C1702-15" value="1N5353" x="7.62" y="-12.065"/>
 <element name="D7" library="diode" package="C1702-15" value="1N5353" x="66.675" y="20.32" rot="R180"/>
 <element name="LED2" library="led" package="LED5MM" value="" x="59.055" y="25.4" rot="R180"/>
@@
 <contactref element="GND" pad="A2"/>
 <contactref element="D7" pad="A"/>
-<contactref element="D5" pad="A"/>
-<contactref element="IC1" pad="IN"/>
-<contactref element="R2" pad="2"/>
-<contactref element="D6" pad="C"/>
-<contactref element="D6" pad="A"/>
-<wire x1="101.6" y1="40.64" x2="107.95" y2="40.64" width="0.8128" layer="16"/>
-<wire x1="101.6" y1="43.4975" x2="101.6" y2="43.18" width="0.8128" layer="16"/>
-<wire x1="97.79" y1="43.4975" x2="101.6" y2="43.4975" width="0.8128" layer="16"/>
-<wire x1="101.6" y1="43.18" x2="101.6" y2="40.64" width="0.8128" layer="16"/>
 <contactref element="LED2" pad="K"/>
 <contactref element="LED3" pad="K"/>
@@
 <vertex x="0" y="0"/>
 </polygon>
-<wire x1="15.24" y1="-12.065" x2="0" y2="-12.065" width="0" layer="19" extent="1-1"/>
-<wire x1="21.59" y1="11.43" x2="15.24" y2="-12.065" width="0" layer="19" extent="1-1"/>
 </signal>
 <signal name="+5V">
@@
 <wire x1="7.62" y1="11.43" x2="11.43" y2="15.24" width="0.8128" layer="16"/>
 </signal>
+<signal name="N$2">
+<contactref element="D5" pad="A"/>
+<contactref element="IC1" pad="IN"/>
+<contactref element="R2" pad="2"/>
+<wire x1="101.6" y1="40.64" x2="107.95" y2="40.64" width="0.8128" layer="16"/>
+<wire x1="101.6" y1="43.4975" x2="101.6" y2="43.18" width="0.8128" layer="16"/>
+<wire x1="97.79" y1="43.4975" x2="101.6" y2="43.4975" width="0.8128" layer="16"/>
+<wire x1="101.6" y1="43.18" x2="101.6" y2="40.64" width="0.8128" layer="16"/>
+</signal>
 </signals>

Commit message: name all the things
Connections:
- net +5V renamed 5V
- net N$1 renamed LED2-P
- net N$10 renamed LED3-P
- net N$11 renamed GATE
- net N$12 renamed LEDP
- net N$13 renamed MISO
- net N$14 renamed SCK
- net N$15 renamed RST
- net N$17 renamed PA3
- net N$18 renamed LED
- net N$19 renamed COLLECTOR
- net N$2 renamed 16V
- net N$20 renamed LVAC2
- net N$21 renamed AUDIO-IN
- net N$22 renamed AUDIO
- net N$23 renamed LVAC1
- net N$24 renamed PA7
- net N$3 renamed PB2
- net N$4 renamed 70VDC
- net N$5 renamed HVDC
- net N$6 renamed PULLUP_DISABLE
- net N$7 renamed RESONANT
- net N$8 renamed PB1
- net N$9 renamed MOSI
Routing:
- net 5V: track 165.4 -> 150.8 mm
